File: hardware/kicad/solar-project/Solar Project.kicad_sch (KiCad schematic)
At the start: 112 parts, among them J1 Solar In, J2 (J_LOG), J3 Battery Bus, J5 Connector,_USB-TYPE-C-16P, M1 IPZ40N, M2 Q_NMOS, M3 Q_NMOS, M4 Q_NMOS, Q1 BSS138, Q2 BSS138, U1 STM32G431CBU6, U2 BSC112N06LD, U3 CP2102-GMR, U4 LM5163DDAR, U5 BSC155N06ND, U6 LM51772QRHARQ1

Commit message: docs: bench-workstation handoff and schematic continuation
Parts:
- removed C28: 100nf, PCM_JLCPCB:C_0805, symbol Device:C
- added C28, C44, C45, C46: 100nF, PCM_JLCPCB:C_0805, symbol PCM_JLCPCB-Capacitors:0805,100nF
- added C30: 47uf, Capacitor_THT:CP_Radial_D6.3mm_P2.50mm, symbol Device:C
- added D8: WS2812B, PCM_JLCPCB:LED-SMD_4P-L1.6-W1.5_XL-1615RGBC-WS2812B, symbol PCM_JLCPCB-Extended:LED, WS2812B, 1615
- added D9: Yellow, PCM_JLCPCB:D_0805, symbol PCM_JLCPCB-Diodes_1:LED,0805,Yellow
- added J4: JTAG, symbol Connector_Generic:Conn_01x04
- added R2: 10Ω, PCM_JLCPCB:R_0805, symbol PCM_JLCPCB-Resistors:0805,10Ω
- added R34: 10kΩ, PCM_JLCPCB:R_0805, symbol PCM_JLCPCB-Resistors_1:0805,10kΩ
- added R44, R45: 4.7kΩ, PCM_JLCPCB:R_0805, symbol PCM_JLCPCB-Resistors:0805,4.7kΩ
- added R46: 330Ω, PCM_JLCPCB:R_0805, symbol PCM_JLCPCB-Resistors:0805,330Ω
- added TP1, TP2, TP3, TP4, TP5: TestPoint_Small, symbol Connector:TestPoint_Small
- added U7: AHT20, AHT20:PSON100P300X300X110-6N, symbol 1My_IC's:AHT20
- added U8: ~, 1My_Parts_ ICs:0.96 inOLED display SSD1306, symbol 1My_Basic components:0.96in_OLED_SSD1306
- D2: value SMBJ64CA -> SMBJ60CA; symbol PCM_JLCPCB-Diodes_1:TVS-Bi,SMBJ64CA -> PCM_JLCPCB-Diodes:TVS-Bi,SMBJ60CA; Category Circuit Protection,ESD And Surge Protection (TVS/ESD) -> TVS/Fuse/Board Level Protection,Electrostatic And Surge Pro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; LCSC C41376099 -> C19077593; Part SMBJ64CA -> SMBJ60CA; Price 0.044USD -> 0.047USD; Stock 9797 -> 36646
- U6: footprint Package_DFN_QFN:Texas_RHA0040B_VQFN-40-1EP_6x6mm_P0.5mm_EP4.15x4.15mm -> RHA0040P-IPC_A
Connections:
- net CHG_OUT_POS: now also TP2.1
- net I2C CLK: now also R44.1, U7.3 (SCL), U8.3 (SLC)
- net I2C DATA: now also R45.1, U7.4 (SDA), U8.4 (SDA)
- net PGND: now also C46.2
- net PV_IN_POS: now also C28.1, TP4.1
- net PWR_NEG: now also C28.2, C30.1, C44.2, C45.2, D8.3 (GND), D9.1, J4.4 (Pin_4), TP5.1, U7.5 (GND), U8.1 (GND), U8.5 (GND), U8.6 (GND), U8.7 (GND), U8.8 (GND)
- net SWCLK: now also J4.1 (Pin_1)
- net SWDIO: now also J4.2 (Pin_2)
- net U6_FLT: now also R34.1
- net U6_VCC2: now also C29.1, C45.1, D8.2 (VDD)
- net VDD: now also C44.1, R34.2, R44.2, R45.2, R46.1, U7.2 (VDD), U8.2 (VCC)
- net V_out: now also C30.2, TP3.1
- net at D5.1, U5.2 (G1), U5.4 (G2): now also R2.1
- net at R16.1, R38.1, U5.5 (D1)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: now also TP1.1
- net at Q1.3 (D), R38.2: now also R2.2
- net at R32.1, U6.16 (ILIMCOMP_ISET), U6.7 (MODE): no longer C29.1
- net at U1.19 (PB2): now also D8.4 (DIN)
- net at C27.1, U6.1 (VCC1): now also C46.1
- new net: D9.2, R46.2
- new net: U7.1 (NC), U7.6 (NC)
- no-connect marks 50 -> 51
Other:
- note added: "DEbugging conn"
- moved on the sheet: C14, D6, D7

Commit message: kicad: sync schematic and cache from local recovery
Parts:
- removed J2: (J_LOG), symbol Connector:Conn_01x03_Pin
- removed TH2: Thermistor_NTC, symbol Device:Thermistor_NTC
- C11, C15, C33, C34, C35, C7, C8: symbol PCM_JLCPCB-Capacitors_1:1206,2.2uF -> PCM_JLCPCB-Capacitors:1206,2.2uF
- C16: footprint SMD,D6.3xL7.7mm -> Capacitor_SMD:CP_Elec_6.3x7.7
- C18, C21: footprint SMD,D10xL12.6mm -> Capacitor_SMD:CP_Elec_10x12.6
- D9: symbol PCM_JLCPCB-Diodes_1:LED,0805,Yellow -> PCM_JLCPCB-Diodes:LED,0805,Yellow
- L3: footprint SMD,7.1x6.6mm -> Inductor_SMD:L_KOHERelec_MDA7030
- M1: footprint TSDSON-8FL -> Package_TO_SOT_SMD:TDSON-8-1
- R14: symbol PCM_JLCPCB-Resistors_1:0805,330kΩ -> PCM_JLCPCB-Resistors:0805,330kΩ
- R15: symbol PCM_JLCPCB-Resistors_1:0805,2kΩ -> PCM_JLCPCB-Resistors:0805,2kΩ
- R36: symbol PCM_JLCPCB-Resistors_1:0805,10kΩ -> PCM_JLCPCB-Resistors:0805,10kΩ
- U4: footprint Package_SO:Texas_R-ESOP-8 -> PCM_JLCPCB:ESOP-8_L4.9-W3.9-P1.27-LS6.0-BL-EP
- U6: footprint RHA0040P-IPC_A -> Package_DFN_QFN:Texas_RHA0040B_VQFN-40-1EP_6x6mm_P0.5mm_EP4.15x4.15mm
Connections:
- net FAULT_OCP: no longer U1.17 (PB0)
- net FAULT_OVP: no longer U1.18 (PB1)
- net CTRL_EN_CHG: no longer names the net of U1.43 (PB5)
- net DRV1: no longer names the net of U6.35 (DRV1)
- net SENSE_TEMP_BOARD: no longer names the net of U1.15 (PA7)
- no-connect marks 51 -> 56
Other:
- note added: "OLED Display"
- note added: "Temp and Humidity sensor Board"
- note added: "UART 1 and power"
- note removed: "Battery Current"
- note removed: "Battery voltage"
- note removed: "Disconnect"
- note removed: "Header (J_LOG)"
- note removed: "Over-Current Protection (FAULT_OCP)"
- note removed: "Over-Voltage Protection (FAULT_OVP)"
- note removed: "PV Current"
- note removed: "PV voltage"
- note removed: "TH_Board"
- note removed: "TH_PWR"
- note removed: "Zone D"
- moved on the sheet: C1, C10, C12, C14, C15, C2, C20, C22, C23, C24, C25, C26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
