File: hardware/kicad/solar-project/Solar Project.kicad_pcb (KiCad board)
At the start: 4 copper layers, 100 x 100.2 mm, 163 parts, among them J1 Solar In, J2 USB4105-GF-A, J3 Battery Bus, J4 JTAG, J5 Fan, M1 IPZ40N, M2 IPZ40N, M3 IPZ40N, M4 IPZ40N, Q1 BSS138, Q2 BSS138, Q3 AO3400A, SW1 Tactile Button, 160gf, SW2 Tactile Button, 160gf, SW3 Tactile Button, 160gf, SW4 Tactile Button, 160gf, SW5 Tactile Button, 160gf, U1 STM32G431CBU6, U10 INA213AIDCKR, U2 BSC112N06LD, U3 CP2102-GMR, U4 LM5163DDAR, U5 BSC155N06ND, U6 LM51772QRHARQ1, U7 AHT20, U9 LMV393, X2 X49SM8MSD2SC

Commit message: Update Rev 0 hardware status and docs
Parts:
- F1: value 10 amp -> Fuse_TD_10A_5x25_63VDC_MIN
- J5: footprint Connector_JST:JST_PH_B3B-PH-K_1x03_P2.00mm_Vertical -> Connector_PinHeader_2.54mm:PinHeader_1x03_P2.54mm_Vertical
- U1: value STM32G431CBU6 -> STM32F411CEU6; footprint Package_DFN_QFN:QFN-48-1EP_6x6mm_P0.4mm_EP4.4x4.4mm_ThermalVias -> Package_DFN_QFN:QFN-48-1EP_7x7mm_P0.5mm_EP5.6x5.6mm
- moved 10mm2 48.9 mm to (170.3, 76.6)
- moved J5 1.04 mm to (195.9, 49.9), turned to 90 degrees
Connections:
- U1 pad 24: unconnected-(U1-PB11-Pad24) -> PWR_NEG
Routing:
- net PWR_NEG: track 291.0 -> 301.2 mm
- net SWCLK: track 22.4 -> 21.2 mm
- net CTRL_3V3: track 354.9 -> 355.9 mm
- net SWDIO: track 15.3 -> 14.5 mm
- net BTN_RT_N: track 80.5 -> 79.8 mm
- net BTN_ENT_N: track 68.2 -> 67.5 mm
- net U6_FLT: track 53.9 -> 53.2 mm
- net Fan Control: track 83.1 -> 82.4 mm
- net V_out _on: track 39.7 -> 39.1 mm
- net TXD: track 19.8 -> 19.3 mm
- net FAULT_OVP: track 66.3 -> 65.7 mm
- net Net-(U1-PF0-OSC_IN): track 21.5 -> 20.9 mm
- net FAULT_OCP: track 54.4 -> 53.8 mm
- net RXD: track 18.7 -> 18.1 mm
- net Net-(S1-A): track 19.4 -> 18.9 mm
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Other:
- board size 100 x 100.2 mm -> 100 x 99.9 mm
- board text added: "+"
- board text added: "-"
- board text added: "Batt Out"
- board text added: "Down"
- board text added: "FAN"
- board text added: "First Build Rev 0"
- board text added: "GND"
- board text added: "I2C Pullups"
- board text added: "Left"
- board text added: "NC"
- board text added: "P Forche"
- board text added: "P Forche TNES LLC 20260723"
- board text added: "PV IN"
- board text added: "Reset"
- board text added: "Right"
- board text added: "SWCLK"
- board text added: "SWDIO"
- board text added: "Solar Charge Controller"
- board text added: "TNES LLC 2026"
- board text added: "UP"
