File: hardware/kicad/solar-project/Solar Project Rev0.kicad_sch (KiCad schematic)
At the start: 167 parts, among them J1 Solar In, J2 USB4105-GF-A, J3 Battery Bus, J4 JTAG, J5 Fan, M1 IPZ40N, M2 IPZ40N, M3 IPZ40N, M4 IPZ40N, Q2 BSS138, Q3 AO3400A, Q4 HSBA0119, Q5 XRS60N10F, Q6 XRS60N10F, SW1 Tactile Button, 160gf, SW2 Tactile Button, 160gf, SW3 Tactile Button, 160gf, SW4 Tactile Button, 160gf, SW5 Tactile Button, 160gf, U1 STM32F411CEU6, U10 INA213AIDCKR, U14 LM74502HDDFR, U3 CP2102-GMR, U4 LM5163DDAR, U6 LM51772QRHARQ1, U7 AHT20, U9 LMV393, X2 X49SM8MSD2SC

Commit message: kicad: split Rev 0 and Rev 1 revision files
Parts:
- removed C52: 100nF, PCM_JLCPCB:C_0805, symbol PCM_JLCPCB-Capacitors:0805,100nF
- removed Q4: HSBA0119, Package_DFN_QFN:PQFN-8-EP_6x5mm_P1.27mm_Generic, symbol Device:Q_PMOS
- removed Q5, Q6: XRS60N10F, Package_DFN_QFN:PQFN-8-EP_6x5mm_P1.27mm_Generic, symbol 1My_Basic components:IPZ40N
- removed R2, R67: 100kΩ, PCM_JLCPCB:R_0805, symbol PCM_JLCPCB-Resistors:0805,100kΩ
- removed R37, R66: 2.2M, PCM_JLCPCB:R_0805, symbol PCM_JLCPCB-Resistors:0805,2.2MΩ
- removed R65: 10Ω, PCM_JLCPCB:R_0805, symbol PCM_JLCPCB-Resistors:0805,10Ω
- removed U14: LM74502HDDFR, Package_TO_SOT_SMD:Texas_DDF0008A_SOT-8_1.6x2.9mm_P0.65mm, symbol 1My_IC's:LM74502HDDFR
- added Q1: BSS138, PCM_JLCPCB:Q_SOT-23, symbol PCM_JLCPCB-Transistors:NMOS,BSS138
- added R2, R39: 10Ω, PCM_JLCPCB:R_0805, symbol PCM_JLCPCB-Resistors:0805,10Ω
- added R37: 100kΩ, PCM_JLCPCB:R_0805, symbol PCM_JLCPCB-Resistors:0805,100kΩ
- added U2: BSC112N06LD, 1My_Parts_ ICs:Infineon_PG-TDSON-8, symbol 1My_Basic components:BSC112N06LD
- added U5: BSC155N06ND, 1My_Parts_ ICs:Infineon_PG-TDSON-8, symbol 1My_Basic components:BSC155N06ND
Connections:
- net CHG_OUT_POS: now also U5.6 (D1)
- net CTRL_3V3: now also R40.1, R37.1
- net PV_IN_POS: now also U2.6 (D1)
- net PV_IN_POS_FUSED: now also U2.5 (D1); no longer D1.1
- net PWR_NEG: now also U1.24 (PB11), Q1.2 (S); no longer R38.2, R40.1
- net V_out _on: now also R39.1; no longer R38.1
- net V_out_sense: now also R38.1, U5.5 (D1)
- net at R42.2: now also D1.1, U2.2 (G1), U2.4 (G2); no longer D1.2
- net at D5.2: now also U5.1 (S1), U5.3 (S2)
- net at J2.A6 (DP1), J2.B6 (DP2): now also D3.3 (I/O2); no longer D3.1 (I/O1)
- net at J2.A7 (DN1), J2.B7 (DN2): now also D3.4 (I/O2); no longer D3.3 (I/O2)
- net at U3.5 (D-): now also D3.6 (I/O1); no longer D3.4 (I/O2)
- net at U3.4 (D+): now also D3.1 (I/O1); no longer D3.6 (I/O1)
- net SRC: no longer names the net of D5.1
- net SRC: now also R2.1, U5.2 (G1), U5.4 (G2)
- new net: Q1.1 (G), R37.2, R39.2
- new net: Q1.3 (D), R2.2, R38.2
- new net: D1.2, U2.1 (S1), U2.3 (S2)
- no-connect marks 45 -> 43
Other:
- moved on the sheet: D1, D3, D5, F2, J2, J3, R24, R42
