File: hardware/kicad/solar-project/Solar Project Rev1.kicad_pcb (KiCad board)
At the start: 4 copper layers, 100 x 99.9 mm, 163 parts, among them J1 Solar In, J2 USB4105-GF-A, J3 Battery Bus, J4 JTAG, J5 Fan, M1 IPZ40N, M2 IPZ40N, M3 IPZ40N, M4 IPZ40N, Q1 BSS138, Q2 BSS138, Q3 AO3400A, SW1 Tactile Button, 160gf, SW2 Tactile Button, 160gf, SW3 Tactile Button, 160gf, SW4 Tactile Button, 160gf, SW5 Tactile Button, 160gf, U1 STM32F411CEU6, U10 INA213AIDCKR, U2 BSC112N06LD, U3 CP2102-GMR, U4 LM5163DDAR, U5 BSC155N06ND, U6 LM51772QRHARQ1, U7 AHT20, U9 LMV393, X2 X49SM8MSD2SC

Commit message: hardware: update Rev1 schematic with 0 ERC errors, BOM, and footprint tables
Parts:
- removed C11: 2.2uF, PCM_JLCPCB:C_1206
- removed C16: 10uf, Capacitor_SMD:CP_Elec_6.3x7.7
- removed C17, C32, C36, C37, C38, C39, C4, C40, C41, C42, C43, C5, C6: 47uf, Capacitor_THT:CP_Radial_D6.3mm_P2.50mm
- removed Q1: BSS138, PCM_JLCPCB:Q_SOT-23
- removed TP3, TP4, TP5: TestPoint_Small, Connector_PinHeader_2.54mm:PinHeader_1x01_P2.54mm_Vertical
- added C52: 100nF, PCM_JLCPCB:C_0805, F.Cu at (229.7, 76.8)
- added C53: 100uF, PCM_JLCPCB:C_1206, F.Cu at (240.1, 98.5)
- added C54: 100nF, PCM_JLCPCB:C_0805, F.Cu at (229.7, 79.8)
- added C55: 1uF, PCM_JLCPCB:C_0805, F.Cu at (229.7, 82.9)
- added C56: 1uF, PCM_JLCPCB:C_0805, F.Cu at (229.7, 85.9)
- added C57: 100nF, PCM_JLCPCB:C_0805, F.Cu at (229.7, 89.0)
- added D10: 1N5819WS, PCM_JLCPCB:D_SOD-323, F.Cu at (229.7, 92.0)
- added D12: Yellow, PCM_JLCPCB:D_0805, F.Cu at (247.9, 99.4)
- added J6: 20021121-00010C4LF, digikey-footprints:PinHeader_2x5_P1.27mm, F.Cu at (249.6, 93.9)
- added Q4: HSBA0119, Package_DFN_QFN:PQFN-8-EP_6x5mm_P1.27mm_Generic, F.Cu at (241.4, 93.4)
- added Q5: BSC040N10NS5, Package_TO_SOT_SMD:TDSON-8-1, F.Cu at (250.2, 78.6)
- added Q6: BSC040N10NS5, Package_TO_SOT_SMD:TDSON-8-1, F.Cu at (250.2, 85.3)
- added Q7: 2N7002K, PCM_JLCPCB:Q_SOT-23, F.Cu at (234.4, 97.2)
- added R65: 10Ω, PCM_JLCPCB:R_0805, F.Cu at (239.5, 76.7)
- added R66: 2.2MΩ, PCM_JLCPCB:R_0805, F.Cu at (239.5, 79.7)
- added R67: 100kΩ, PCM_JLCPCB:R_0805, F.Cu at (239.5, 82.6)
- added R68: 1.3k, PCM_JLCPCB:R_0805, F.Cu at (239.5, 85.6)
- added R69: 10Ω, PCM_JLCPCB:R_0805, F.Cu at (239.5, 88.5)
- added R70: 10Ω, PCM_JLCPCB:R_0805, F.Cu at (243.9, 76.7)
- added R71: 10Ω, PCM_JLCPCB:R_0805, F.Cu at (243.9, 79.7)
- added R72: 10Ω, PCM_JLCPCB:R_0805, F.Cu at (243.9, 82.6)
- added R73: 10Ω, PCM_JLCPCB:R_0805, F.Cu at (243.9, 85.6)
- added R74: 100kΩ, PCM_JLCPCB:R_0805, F.Cu at (243.9, 88.5)
- added TP15: 5015, TestPoint:TestPoint_Keystone_5015_Micro_Mini, F.Cu at (234.6, 77.1)
- added TP16: 5015, TestPoint:TestPoint_Keystone_5015_Micro_Mini, F.Cu at (234.6, 80.9)
- added TP17: 5015, TestPoint:TestPoint_Keystone_5015_Micro_Mini, F.Cu at (234.6, 84.6)
- added TP18: 5015, TestPoint:TestPoint_Keystone_5015_Micro_Mini, F.Cu at (234.6, 88.4)
- added U14: LM74502HDDFR, Package_TO_SOT_SMD:Texas_DDF0008A_SOT-8_1.6x2.9mm_P0.65mm, F.Cu at (234.6, 92.6)
- C18: value 560uf -> 560uF
- C19, C30: value 47uf -> 47uF; footprint Capacitor_THT:CP_Radial_D6.3mm_P2.50mm -> Capacitor_THT:C_Radial_D8.0mm_H7.0mm_P3.50mm
- C20: value 180pf -> 180pF
- C21: value 560uf -> 47uF; footprint Capacitor_SMD:CP_Elec_10x12.6 -> Capacitor_THT:C_Radial_D8.0mm_H7.0mm_P3.50mm
- C23: value 100nf -> 100nF
- C24: value 220nf -> 22nF
- C25: value 1.5nf -> 1.5nF
- C26: value 33nf -> 33nF
- C3: value 47uf -> 100uF
- C31: value 47uf -> 47uF; footprint Capacitor_THT:CP_Radial_D6.3mm_P2.50mm -> Capacitor_THT:CP_Radial_D8.0mm_P3.50mm
- C33, C8: value 2.2uF -> 100nF; footprint PCM_JLCPCB:C_1206 -> PCM_JLCPCB:C_0805
- D9: value Yellow -> Green
- F1: value Fuse_TD_10A_5x25_63VDC_MIN -> Fuse
- J1: value Solar In -> Screw_Terminal_01x02
- J3: value Battery Bus -> Screw_Terminal_01x02
- J4: value JTAG -> Conn_01x04
- J5: value Fan -> Conn_01x03_Socket
- L2: value 1uh -> L; footprint 1My_Parts_ Passive:HC3-1R0-R -> Inductor_SMD:L_APV_APH1240
- L3: value 68uh -> L
- M1, M2, M3, M4: value IPZ40N -> CSD18540Q5B
- Q2: value BSS138 -> 2N7002K
- Q3: value AO3400A -> 2N7002K
- R10: value 22kΩ -> 20kΩ
- R11: value 240k -> 330Ω
- R16: footprint 1My_Parts_ Passive:R_2512 Shunt 4 pad resistor -> Resistor_SMD:R_Shunt_Vishay_WSK2512_6332Metric_T2.66mm
- R18, R3: value 66.5k -> 76.8k
- R2: value 10Ω -> 100kΩ
- R20: value 499kΩ -> 499k
- R28: footprint PCM_JLCPCB:R_0603 -> PCM_JLCPCB:R_0805
- R31: value 2.43K -> 2.43k
- R33: value 6.49k -> 0Ω
- R37: value 100kΩ -> 2.2MΩ
- R39: value 10Ω -> 330Ω
- R42: value 10Ω -> 1kΩ
- R46: value 330Ω -> 82kΩ
- R6: value 22kΩ -> 10kΩ
- R7: value 430k -> 20kΩ
- U1: value STM32F411CEU6 -> STM32G431CBU6
- U2: value BSC112N06LD -> ESP32_C3_mini; footprint 1My_Parts_ ICs:Infineon_PG-TDSON-8 -> 1My_Parts_ MPUs:ESP32 C3 mini
- U4: value LM5163DDAR -> LM5163
- U5: value BSC155N06ND -> LP5912-3.3DRV; footprint 1My_Parts_ ICs:Infineon_PG-TDSON-8 -> Package_SON:WSON-6-1EP_2x2mm_P0.65mm_EP1x1.6mm_ThermalVias
- U6: footprint Package_DFN_QFN:Texas_RHA0040B_VQFN-40-1EP_6x6mm_P0.5mm_EP4.15x4.15mm -> digikey-footprints:VFQFN-40-1EP_6x6mm
- U8: value ~ -> SSD1306_OLED
- moved M2 72.9 mm to (78.3, 114.2)
- moved M1 56.7 mm to (85.7, 79.9)
- moved L2 56.4 mm to (88.6, 100.0), turned to 0 degrees
- moved R22 39.6 mm to (111.3, 90.1)
Connections:
- C14 pad 1: CTRL_3V3 -> CTRL_5V
- C21 pad 1: V_out -> PV_IN_POS
- C25 pad 1: PGND -> PWR_NEG
- C26 pad 1: PGND -> PWR_NEG
- C27 pad 2: PGND -> PWR_NEG
- C30 pad 1: V_out -> PV_IN_POS
- C31 pad 1: V_out -> PV_IN_POS
- C33 pad 1: V_out -> PWR_NEG
- C33 pad 2: PWR_NEG -> V_out
- C46 pad 2: PGND -> PWR_NEG
- C8 pad 1: PWR_NEG -> PV_IN_POS
- C8 pad 2: PV_IN_POS -> PWR_NEG
- C9 pad 1: CTRL_3V3 -> CTRL_5V
- D1 pad 1: Net-(U2-G1) -> /PV_IN_POS_FUSED
- D1 pad 2: Net-(U2-S1) -> Net-(D1-Pad2)
- D3 pad 1: Net-(U3-D+) -> Net-(J2-DP1)
- D3 pad 3: Net-(J2-DP1) -> Net-(J2-DN1)
- D3 pad 4: Net-(J2-DN1) -> Net-(U3-D-)
- D3 pad 6: Net-(U3-D-) -> Net-(U3-D+)
- D5 pad 1: Net-(U5-G1) -> SRC
- D5 pad 2: Net-(U5-S1) -> Net-(Q5-G)
- D8 pad 2: U6_VCC2 -> CTRL_5V
- L2 pad 1: _CSB_2 -> Net-(L2-Pad1)
- L3 pad 2: CTRL_3V3 -> CTRL_5V
- R10 pad 2: CTRL_3V3 -> CTRL_5V
- R11 pad 1: PWR_NEG -> CTRL_5V
- R11 pad 2: Net-(R11-Pad2) -> Net-(D9-Pad2)
- R16 pad 1: V_out_sense -> V_out
- R16 pad 2: V_out_sense -> V_out_SNS_P 
- R16 pad 3: V_out -> V_out_SNS_N
- R16 pad 4: V_out -> V_out_sense
- R2 pad 1: Net-(U5-G1) -> SRC
- R2 pad 2: Net-(Q1-D) -> Net-(Q5-G)
- R22 pad 1: _CSB_2 -> Net-(L2-Pad1)
- R22 pad 3: SW_1 -> _CSA_2
- R26 pad 1: SW_1 -> _CSA_2
- R28 pad 2: PGND -> PWR_NEG
- R29 pad 2: PGND -> PWR_NEG
- R30 pad 2: PGND -> PWR_NEG
- R31 pad 2: PGND -> PWR_NEG
- R32 pad 1: Net-(U6-ILIMCOMP_ISET) -> U6_VCC2
- R32 pad 2: PWR_NEG -> Net-(U6-MODE)
- R33 pad 2: PGND -> PWR_NEG
- R34 pad 1: U6_FLT -> CTRL_3V3
- R34 pad 2: CTRL_3V3 -> U6_FLT
- R37 pad 1: CTRL_3V3 -> V_out_sense
- R37 pad 2: Net-(Q1-G) -> Net-(R37-Pad2)
- R38 pad 1: V_out_sense -> V_out _on
- R38 pad 2: Net-(Q1-D) -> PWR_NEG
- R39 pad 1: V_out _on -> CTRL_3V3
- R39 pad 2: Net-(Q1-G) -> Net-(D12-Pad2)
- R40 pad 1: CTRL_3V3 -> PWR_NEG
- R42 pad 2: Net-(U2-G1) -> Net-(D1-Pad2)
- R46 pad 1: CTRL_3V3 -> Net-(R46-Pad1)
- R46 pad 2: Net-(D9-Pad2) -> PWR_NEG
- R6 pad 1: Net-(R11-Pad2) -> PWR_NEG
- R63 pad 2: V_out_sense -> V_out_SNS_N
- R64 pad 2: V_out -> V_out_SNS_P 
- U1 pad 14: unconnected-(U1-PA6-Pad14) -> CTS
- U1 pad 15: unconnected-(U1-PA7-Pad15) -> RTS
- U1 pad 22: unconnected-(U1-PB10-Pad22) -> CTS_ESP
- U1 pad 24: PWR_NEG -> RTS_ESP
- U1 pad 25: unconnected-(U1-PB12-Pad25) -> CTRL_EN_CHG
- U1 pad 33: CTS -> RXD_ESP
- U1 pad 34: RTS -> TXD_ESP
- U10 pad 4: V_out -> V_out_SNS_P 
- U10 pad 5: V_out_sense -> V_out_SNS_N
- U2 pad 1: Net-(U2-S1) -> unconnected-(U2-GPIO5-Pad1)
- U2 pad 2: Net-(U2-G1) -> unconnected-(U2-GPIO6-Pad2)
- U2 pad 3: Net-(U2-S1) -> unconnected-(U2-GPIO7-Pad3)
- U2 pad 4: Net-(U2-G1) -> unconnected-(U2-GPIO8-Pad4)
- U2 pad 5: /PV_IN_POS_FUSED -> unconnected-(U2-GPIO9-Pad5)
- U2 pad 6: PV_IN_POS -> unconnected-(U2-GPIO10-Pad6)
- U5 pad 1: Net-(U5-S1) -> CTRL_3V3
- U5 pad 2: Net-(U5-G1) -> unconnected-(U5-NC-Pad2)
- U5 pad 3: Net-(U5-S1) -> unconnected-(U5-PG-Pad3)
- U5 pad 4: Net-(U5-G1) -> CTRL_5V
- U5 pad 5: V_out_sense -> PWR_NEG
- U5 pad 6: CHG_OUT_POS -> CTRL_5V
- U6 pad 24: HO1 -> Net-(U6-HO1)
- U6 pad 27: LO1 -> Net-(U6-LO1)
- U6 pad 28: PGND -> PWR_NEG
- U6 pad 30: LO2 -> Net-(U6-LO2)
- U6 pad 32: HO2 -> Net-(U6-HO2)
- U6 pad 7: Net-(U6-ILIMCOMP_ISET) -> Net-(U6-MODE)
Routing:
- net CTRL_3V3: track 355.9 -> 0.00 mm, vias 16 -> 0
- net PWR_NEG: track 301.2 -> 0.00 mm, vias 140 -> 0
- net PV_IN_POS: track 274.5 -> 0.00 mm
- net V_out: track 191.8 -> 0.00 mm, vias 3 -> 0
- net V_in_ADC: track 146.3 -> 0.00 mm, vias 3 -> 0
- net CHG_OUT_POS: track 140.4 -> 0.00 mm, vias 6 -> 0
- net SW_1: track 138.1 -> 0.00 mm, vias 6 -> 0
- net BAT_BUS_POS: track 137.7 -> 0.00 mm, vias 4 -> 0
- net V_in_ON: track 134.2 -> 0.00 mm, vias 4 -> 0
- net I2C DATA: track 109.4 -> 0.00 mm, vias 4 -> 0
- net VBUS: track 108.9 -> 0.00 mm, vias 5 -> 0
- net I2C CLK: track 108.1 -> 0.00 mm, vias 4 -> 0
- net Fan Control: track 82.4 -> 0.00 mm, vias 4 -> 0
- net BTN_RT_N: track 79.8 -> 0.00 mm, vias 2 -> 0
- net U6_VCC2: track 75.8 -> 0.00 mm, vias 2 -> 0
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
Commit message: handoff: save local Rev1 work for laptop
Parts:
- removed J5: Conn_01x03_Socket, Connector_PinHeader_2.54mm:PinHeader_1x03_P2.54mm_Vertical
- added J7: Fan, Connector_PinHeader_2.54mm:PinHeader_1x03_P2.54mm_Vertical, F.Cu at (221.1, 47.3)
- F1, F2: value Fuse -> 3522-2
- moved TP17 115.7 mm to (127.5, 128.2)
- moved TP18 115.7 mm to (127.5, 132.0)
- moved Q4 108.7 mm to (135.2, 70.3)
- moved TP1 103.6 mm to (257.3, 131.9)
- moved 10mm1 103.6 mm to (306.7, 142.2)
- moved C54 101.9 mm to (135.9, 119.3)
- moved C55 101.9 mm to (135.9, 122.4)
- moved C56 101.9 mm to (135.9, 125.4)
- moved TP16 100.3 mm to (139.3, 49.7)
- moved D12 99.0 mm to (149.9, 113.3)
- moved C53 98.6 mm to (145.2, 125.2)
- moved D10 96.1 mm to (140.3, 127.1)
- moved C57 94.0 mm to (167.7, 18.3)
- moved J6 90.7 mm to (159.8, 81.4)
- moved C3 89.5 mm to (187.1, 56.7)
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Connections:
- D1 pad 2: Net-(D1-Pad2) -> Net-(Q4-G)
- D8 pad 1: unconnected-(D8-DOUT-Pad1) -> Net-(D11-DIN)
- F1 pad 2: /PV_IN_POS_RAW -> /PV_IN_POS_FUSED
- F2 pad 1: CHG_OUT_POS -> BAT_BUS_POS
- Q4 pad 1: (no net) -> /PV_IN_POS_FUSED
- Q4 pad 2: (no net) -> /PV_IN_POS_FUSED
- Q4 pad 3: (no net) -> unconnected-(Q4-S-Pad3)
- Q4 pad 4: (no net) -> Net-(Q4-G)
- Q4 pad 5: (no net) -> PV_IN_POS
- Q6 pad 1: CHG_OUT_POS -> SRC
- Q6 pad 2: CHG_OUT_POS -> SRC
- Q6 pad 3: CHG_OUT_POS -> SRC
- Q6 pad 5: SRC -> CHG_OUT_POS
- R42 pad 2: Net-(D1-Pad2) -> Net-(Q4-G)
- U1 pad 3: BTN_RT_N -> unconnected-(U1-PC14-OSC32_IN-Pad3)
- U1 pad 39: unconnected-(U1-PC10-Pad39) -> BTN_RT_N
- U1 pad 43: unconnected-(U1-PB5-Pad43) -> FAN_TACH
Routing:
- net /PV_IN_POS_RAW: track 0.00 -> 13.6 mm
- added copper zone on F.Cu, net Net-(L2-Pad1)
- added copper zone on F.Cu, net PV_IN_POS
- added copper zone on F.Cu, net SRC
- removed copper zone on F.Cu, net CHG_OUT_POS
- removed copper zone on F.Cu, net _CSB_2
