File: hardware/kicad/solar-project/Solar Project Rev1.kicad_pcb (KiCad board)
At the start: 4 copper layers, 100 x 99.9 mm, 172 parts, among them J1 Screw_Terminal_01x02, J2 USB4105-GF-A, J3 Screw_Terminal_01x02, J4 Conn_01x04, J6 20021121-00010C4LF, J7 Fan, M1 CSD18540Q5B, M2 CSD18540Q5B, M3 CSD18540Q5B, M4 CSD18540Q5B, Q2 2N7002K, Q3 2N7002K, Q4 HSBA0119, Q5 BSC040N10NS5, Q6 BSC040N10NS5, Q7 2N7002K, SW1 Tactile Button, 160gf, SW2 Tactile Button, 160gf, SW3 Tactile Button, 160gf, SW4 Tactile Button, 160gf, SW5 Tactile Button, 160gf, U1 STM32G431CBU6, U10 INA213AIDCKR, U14 LM74502HDDFR, U2 ESP32_C3_mini, U3 CP2102-GMR, U4 LM5163, U5 LP5912-3.3DRV, U6 LM51772QRHARQ1, U7 AHT20, U8 SSD1306_OLED, U9 LMV393, X2 X49SM8MSD2SC

Commit message: Save local changes: snapshot of docs, KiCad Rev1, BOM and hardware files
Parts:
- added D11: WS2812B, PCM_JLCPCB:LED-SMD_4P-L1.6-W1.5_XL-1615RGBC-WS2812B, F.Cu at (165.7, 115.8)
- C19, C21, C30: footprint Capacitor_THT:C_Radial_D8.0mm_H7.0mm_P3.50mm -> Capacitor_THT:CP_Radial_D8.0mm_P3.50mm
- F1, F2: footprint Fuse:Fuseholder_Littelfuse_100_series_5x25mm -> 1My_Parts_ Passive:Automotive fuse holder keystone 3522-2_KEY
- moved C57 122.0 mm to (167.4, 140.3), turned to 90 degrees
- moved U2 113.9 mm to (169.0, 133.5), turned to 180 degrees
- moved U8 112.5 mm to (134.8, 118.8)
- moved 10mm1 112.2 mm to (214.3, 78.5)
- moved TP15 76.4 mm to (142.1, 140.5)
- moved TP1 55.7 mm to (216.2, 94.2)
- moved D8 52.8 mm to (165.7, 112.4)
- moved X2 44.8 mm to (181.2, 100.3), turned to 180 degrees
- moved C50 42.7 mm to (180.6, 105.5), turned to 180 degrees
- moved R45 38.6 mm to (189.7, 105.5)
- moved R44 36.9 mm to (185.1, 105.5)
- moved C49 34.8 mm to (175.1, 105.5), turned to 0 degrees
- moved Q3 33.1 mm to (198.4, 50.6), turned to 90 degrees
- moved R4 31.4 mm to (198.4, 57.3), turned to 180 degrees
- moved R39 30.8 mm to (158.1, 137.4)
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Connections:
- D1 pad 1: /PV_IN_POS_FUSED -> Net-(D1-Pad1)
- D2 pad 2: /PV_IN_POS_FUSED -> Net-(D1-Pad1)
- F1 pad 1: /PV_IN_POS_FUSED -> Net-(D1-Pad1)
- F1 pad 2: /PV_IN_POS_FUSED -> Net-(D1-Pad1)
- J1 pad 1: /PV_IN_POS_RAW -> Net-(J1-Pin_1)
- Q4 pad 1: /PV_IN_POS_FUSED -> Net-(D1-Pad1)
- Q4 pad 2: /PV_IN_POS_FUSED -> Net-(D1-Pad1)
- Q4 pad 3: unconnected-(Q4-S-Pad3) -> Net-(D1-Pad1)
- R35 pad 1: /PV_IN_POS_FUSED -> Net-(D1-Pad1)
- R43 pad 1: /PV_IN_POS_FUSED -> Net-(D1-Pad1)
Routing:
- net PWR_NEG: track 0.00 -> 743.4 mm, vias 0 -> 53
- net CTRL_3V3: track 0.00 -> 354.3 mm, vias 0 -> 14
- net PV_IN_POS: track 0.00 -> 168.7 mm, vias 0 -> 12
- net CTRL_5V: track 0.00 -> 135.7 mm, vias 0 -> 7
- net I2C DATA: track 0.00 -> 123.1 mm, vias 0 -> 4
- net _Undervoltage Feedback: track 0.00 -> 107.8 mm, vias 0 -> 4
- net BAT_BUS_POS: track 0.00 -> 103.9 mm, vias 0 -> 3
- net VBUS: track 0.00 -> 100.9 mm, vias 0 -> 3
- net CHG_OUT_POS: track 0.00 -> 100.3 mm, vias 0 -> 6
- net I2C CLK: track 0.00 -> 99.6 mm, vias 0 -> 4
- net V_in_ADC: track 0.00 -> 78.9 mm, vias 0 -> 3
- net _OUTPUT Feedback: track 0.00 -> 77.5 mm, vias 0 -> 3
- net V_out_sense: track 0.00 -> 70.2 mm, vias 0 -> 3
- net FAN_TACH: track 0.00 -> 69.3 mm, vias 0 -> 1
- net Fan Control: track 0.00 -> 65.9 mm, vias 0 -> 2
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- added copper zone on F.Cu, net CHG_OUT_POS
- added copper zone on F.Cu, net Net-(D1-Pad1)
- removed copper zone on F.Cu, net /PV_IN_POS_FUSED
- removed copper zone on F.Cu, net V_out_sense
Other:
- board text added: "3.3V"
- board text added: "5V"
- board text added: "Build : Rev 1"
- board text added: "MPPT Charge Controller"
- board text added: "P Forche TNES LLC 20260915"
- board text added: "System"
- board text added: "WIFI"
- board text removed: "F2"
- board text removed: "First Build Rev 0"
- board text removed: "I2C Pullups"
- board text removed: "P Forche TNES LLC 20260723"
- board text removed: "Solar Charge Controller"

Commit message: Rev1: close Track E PCB layout (routed, DRC clean, JLCPCB DFM pass), clean up duplicate LCSC schematic fields, close Track B/C docs, add fab outputs
- DEC-064: remove 172 duplicate empty 'LCSC ' (trailing-space) properties from Solar Project Rev1.kicad_sch; ERC warnings 337 -> 171, only field_name_whitespace category changed
- DEC-065: Track E closed - board fully routed (4-layer), DRC 0 errors/0 unconnected, JLCPCB DFM check passed; fab-ready Gerbers/drill archived under hardware/kicad/solar-project/fab-output-2026-09-18/
- Update rev-one-closure-plan-2026-09-16.md: Track A/B/C/E status banners, Section 0 path-to-order summary, Section 3/4 sequencing refreshed
- Update decisions-log.md through DEC-065
- Carry forward Track B BOM/order-guide reconciliation and DEC-063 closure from 2026-09-17
- Add SOLAR_HANDOFF_2026-09-18.md and update NEXT_CHAT_PROMPT.md to point next session at Track D (Rev 0 evidence mining)
Parts:
- added J8: Conn_01x04, Connector_PinHeader_2.54mm:PinHeader_1x04_P2.54mm_Vertical, F.Cu at (217.0, 85.0)
- C52: value 100nF -> 220nF
- D2: value SMBJ60CA -> SMBJ48CA
- moved TP1 3.55 mm to (215.3, 97.6)
- moved 10mm1 0.46 mm to (213.9, 78.8)
Routing:
- net I2C CLK: track 99.6 -> 136.8 mm
- net I2C DATA: track 123.1 -> 156.1 mm, vias 4 -> 5
- net CTRL_3V3: track 354.3 -> 377.0 mm
- net PWR_NEG: track 743.4 -> 750.2 mm
- net PV_IN_POS: track 168.7 -> 164.0 mm
