File: hardware/kicad/solar-project/Solar Project Rev1.kicad_sch (KiCad schematic)
At the start: 167 parts, among them J1 Solar In, J2 USB4105-GF-A, J3 Battery Bus, J4 JTAG, J5 Fan, M1 IPZ40N, M2 IPZ40N, M3 IPZ40N, M4 IPZ40N, Q2 BSS138, Q3 AO3400A, Q4 HSBA0119, Q5 XRS60N10F, Q6 XRS60N10F, SW1 Tactile Button, 160gf, SW2 Tactile Button, 160gf, SW3 Tactile Button, 160gf, SW4 Tactile Button, 160gf, SW5 Tactile Button, 160gf, U1 STM32F411CEU6, U10 INA213AIDCKR, U14 LM74502HDDFR, U3 CP2102-GMR, U4 LM5163DDAR, U6 LM51772QRHARQ1, U7 AHT20, U9 LMV393, X2 X49SM8MSD2SC

Commit message: docs: Rev0 bring-up addendum, revision labeling, bench plan updates
- Add Rev 0 bench addendum for missing M1-M4 bridge MOSFETs (footprint mismatch)
- Rebuild Rev 1 bench bring-up plan with staged safety gates
- Add REVISION-INDEX.md to disambiguate Rev 0 manufactured vs Rev 1 active files
- Rename generic Solar Project.* files to explicit Rev1/dated snapshot names
- Ignore all KiCad lock file variants (~*.lck)
Parts:
- removed R11: 240k, PCM_JLCPCB:R_0805, symbol Device:R
- removed R46: 330Ω, PCM_JLCPCB:R_0805, symbol PCM_JLCPCB-Resistors:0805,330Ω
- added C53: 100uF, PCM_JLCPCB:C_1206, symbol PCM_JLCPCB-Capacitors:1206,100uF
- added C54, C57: 100nF, PCM_JLCPCB:C_0805, symbol PCM_JLCPCB-Capacitors:0805,100nF
- added C55, C56: 1uF, PCM_JLCPCB:C_0805, symbol PCM_JLCPCB-Capacitors:0805,1uF
- added D10: 1N5819WS, PCM_JLCPCB:D_SOD-323, symbol PCM_JLCPCB-Diodes:Schottky,1N5819WS
- added D12: Yellow, PCM_JLCPCB:D_0805, symbol PCM_JLCPCB-Diodes:LED,0805,Yellow
- added R11, R39: 330Ω, PCM_JLCPCB:R_0805, symbol PCM_JLCPCB-Resistors:0805,330Ω
- added U2: ESP32_C3_mini, 113991054:MODULE_113991054, symbol 1My_MPUs:ESP32_C3_mini
- added U5: LP5912-3.3DRV, Package_SON:WSON-6-1EP_2x2mm_P0.65mm_EP1x1.6mm_ThermalVias, symbol Regulator_Linear:LP5912-3.3DRV
- D9: value Yellow -> Green; symbol PCM_JLCPCB-Diodes:LED,0805,Yellow -> PCM_JLCPCB-Diodes:LED,0805,Green; Category Optocouplers & LEDs & Infrared,Light Emitting Diodes (LED) -> Optoelectronics,Light Emitting Diodes (LED); Emitted Color Yellow -> Emerald; LCSC C2296 -> C2297; Part KT-0805Y -> KT-0805G; Price 0.015USD -> 0.014USD; Stock 662678 -> 2062782
- R10: value 22kΩ -> 20kΩ; symbol PCM_JLCPCB-Resistors:0805,22kΩ -> PCM_JLCPCB-Resistors:0805,20kΩ; LCSC C17560 -> C4328; Part 0805W8F2202T5E -> 0805W8F2002T5E; Resistance 22kΩ -> 20kΩ; Stock 534855 -> 1613783
- R6: value 22kΩ -> 10kΩ; symbol PCM_JLCPCB-Resistors:0805,22kΩ -> PCM_JLCPCB-Resistors:0805,10kΩ; LCSC C17560 -> C17414; Part 0805W8F2202T5E -> 0805W8F1002T5E; Resistance 22kΩ -> 10kΩ; Stock 534855 -> 12301172
- R7: value 430k -> 20kΩ; symbol PCM_JLCPCB-Resistors:0805,49.9kΩ -> PCM_JLCPCB-Resistors:0805,20kΩ; Attrition Qty (none) -> 10; Category (none) -> Resistors,Chip Resistor - Surface Mount; Class (none) -> Basic Component; LCSC C865487 -> C4328; Manufacturer (none) -> UNI-ROYAL(Uniroyal Elec); Minimum Qty (none) -> 20; Operating Temperature Range (none) -> -55°C~+155°C; Overload Voltage (Max) (none) -> 150V; Part (none) -> 0805W8F2002T5E; Power(Watts) (none) -> 125mW; Price (none) -> 0.005USD; Process (none) -> SMT; Resistance (none) -> 20kΩ; Stock (none) -> 1613783; Temperature Coefficient (none) -> ±100ppm/°C; Tolerance (none) -> ±1%; Type (none) -> Thick Film Resistors
Connections:
- net CTRL_3V3: now also C53.1, C54.1, C55.1, R39.1, U5.1 (OUT); no longer C14.1, C9.1, L3.2, R10.2
- net CTS: now also U1.14 (PA6); no longer U1.33 (PA11)
- net PWR_NEG: now also R6.1, C53.2, C54.2, C55.2, C56.2, C57.2, D12.1, U2.15 (GND), U5.5 (GND), U5.7 (EP)
- net RTS: now also U1.15 (PA7); no longer U1.34 (PA12)
- net VBUS: now also D10.2
- net CTS_ESP: now reaches U1.22 (PB10)
- net CTS_ESP: now also U2.7 (GPIO20)
- net RTS_ESP: now reaches U1.24 (PB11)
- net RTS_ESP: now also U2.8 (GPIO21)
- net at D9.2: now also R11.2
- new net: D12.2, R39.2
- new net CTRL_5V: C14.1, C56.1, C57.1, C9.1, D10.1, L3.2, R10.2, R11.1, U2.16 (5V), U5.4 (EN), U5.6 (IN)
- new net RXD_ESP: U1.33 (PA11), U2.9 (GPIO0)
- new net TXD_ESP: U1.34 (PA12), U2.10 (GPIO1)
- no-connect marks 45 -> 52
Other:
- note added: "5 Volt Buck"
- note removed: "3.3V control"
- moved on the sheet: C10, C14, C15, D4, D6, D7, D9, L2, L3, R10, R12, R13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

Commit message: Rebaseline Rev 1 converter design
Parts:
- removed C11, C33, C8: 2.2uF, PCM_JLCPCB:C_1206, symbol PCM_JLCPCB-Capacitors:1206,2.2uF
- removed C16: 10uf, Capacitor_SMD:CP_Elec_6.3x7.7, symbol Device:C
- removed C17, C31, C32, C36, C37, C38, C39, C4, C40, C41, C42, C43, C5, C6: 47uf, Capacitor_THT:CP_Radial_D6.3mm_P2.50mm, symbol Device:C
- removed M1: IPZ40N, Package_TO_SOT_SMD:TDSON-8-1, symbol 1My_Basic components:IPZ40N
- added C33, C8: 100nF, PCM_JLCPCB:C_0805, symbol PCM_JLCPCB-Capacitors:0805,100nF
- added M1: CSD18540Q5B, Package_TO_SOT_SMD:TDSON-8-1, symbol Transistor_FET:CSD18540Q5B
- added TP10, TP11, TP6, TP7, TP8, TP9: TestPoint_Small, Connector_PinHeader_2.54mm:PinHeader_1x01_P2.54mm_Vertical, symbol Connector:TestPoint_Small
- 10mm1, 10mm2, U8: value ~ -> (none)
- C19, C30: footprint Capacitor_THT:CP_Radial_D6.3mm_P2.50mm -> Through Hole,D8xL11.5mm; LCSC C122243 -> C44606514
- C21: value 560uf -> 47uf; footprint Capacitor_SMD:CP_Elec_10x12.6 -> Through Hole,D8xL11.5mm; LCSC C264031 -> C44606514
- C26: value 33nf -> 10uf
- C3: value 47uf -> 100uf; LCSC C122243 -> C49232871
- C7: value 2.2uF -> 1uf 100v; footprint PCM_JLCPCB:C_1206 -> PCM_JLCPCB:C_0805; Attrition Qty 8 -> (none); Capacitance 2.2uF -> (none); Category Capacitors,Multilayer Ceramic Capacitors MLCC - SMD/SMT -> (none); Class Basic Component -> (none); LCSC C50254 -> C6119946; Manufacturer Samsung Electro-Mechanics -> (none); Minimum Qty 5 -> (none); Part CL31B225KBHNNNE -> (none); Price 0.032USD -> (none); Process SMT -> (none); Stock 180873 -> (none); Temperature Coefficient X7R -> (none); Tolerance ±10% -> (none); Voltage Rated 50V -> (none)
- L2: value 1uh -> 3.3uh; footprint 1My_Parts_ Passive:HC3-1R0-R -> Inductor_SMD:L_APV_APH1240; LCSC  (none) -> C49308530
- M2, M3, M4: value IPZ40N -> CSD18540Q5B; symbol 1My_Basic components:IPZ40N -> Transistor_FET:CSD18540Q5B; LCSC C6969335 -> C86513
- Q2: value BSS138 -> 2N7002K; symbol PCM_JLCPCB-Transistors:NMOS,BSS138 -> PCM_JLCPCB-Transistors:NMOS,2N7002K; Attrition Qty 5 -> 4; Continuous Drain Current (Id) 340mA -> (none); Drain Source On Resistance (RDS(on)@Vgs,Id) 2.5Ω@10V,0.34A -> (none); Drain Source Voltage (Vdss) null -> (none); Gate Threshold Voltage (Vgs(th)@Id) 1.6V@250uA -> (none); Input Capacitance (Ciss@Vds) 17.5pF@25V -> (none); LCSC C7420339 -> C22379475; Operating Temperature -55°C~+150°C -> (none); Part BSS138 -> 2N7002K; Power Dissipation (Pd) 350mW -> (none); Price 0.021USD -> 0.019USD; Reverse Transfer Capacitance (Crss@Vds) 6.5pF@25V -> (none); Stock 257620 -> 82639; Total Gate Charge (Qg@Vgs) 1.7nC@10V -> (none); Type null -> (none)
- Q3: value AO3400A -> 2N7002K; symbol PCM_JLCPCB-Transistors:NMOS,AO3400A -> PCM_JLCPCB-Transistors:NMOS,2N7002K; Category Transistors,MOSFETs -> Triode/MOS Tube/Transistor,MOSFETs; Class Basic Component -> Preferred Component; Continuous Drain Current (Id) 5.7A -> (none); Drain Source On Resistance (RDS(on)@Vgs,Id) 26.5mΩ@10V,5.7A -> (none); Drain Source Voltage (Vdss) 30V -> (none); Gate Threshold Voltage (Vgs(th)@Id) 1.5V@250uA -> (none); Input Capacitance (Ciss@Vds) 630pF@15V -> (none); LCSC C20917 -> C22379475; Manufacturer Alpha & Omega Semicon -> hongjiacheng; Minimum Qty 5 -> 10; Operating Temperature -55°C~+150°C@(Tj) -> (none); Part AO3400A -> 2N7002K; Power Dissipation (Pd) 1.4W -> (none); Price 0.074USD -> 0.019USD; Stock 463122 -> 82639; Total Gate Charge (Qg@Vgs) 7nC@4.5V -> (none); Type 1 N-channel -> (none)
- Q5: value XRS60N10F -> CSD18563Q5A; footprint Package_DFN_QFN:PQFN-8-EP_6x5mm_P1.27mm_Generic -> Package_TO_SOT_SMD:TDSON-8-1; symbol 1My_Basic components:IPZ40N -> Transistor_FET:CSD18563Q5A; LCSC C42457069 -> C86513
- Q6: value XRS60N10F -> CSD18563Q5A; footprint Package_DFN_QFN:PQFN-8-EP_6x5mm_P1.27mm_Generic -> Package_TO_SOT_SMD:TDSON-8-1; symbol 1My_Basic components:IPZ40N -> Transistor_FET:CSD18563Q5A; LCSC (none) -> C86513
- R16: footprint 1My_Parts_ Passive:R_2512 Shunt 4 pad resistor -> Resistor_SMD:R_Shunt_Vishay_WSK2512_6332Metric_T2.66mm
- R18: value 66.5k -> 76.8k; LCSC C2090706 -> (none); LCSC  (none) -> C3000581
- R3: value 66.5k -> 76.8k; LCSC  (none) -> C3000581
- R33: value 6.49k -> 0Ω; symbol Device:R -> PCM_JLCPCB-Resistors:0805,0Ω; Attrition Qty (none) -> 10; Category (none) -> Resistors,Chip Resistor - Surface Mount; Class (none) -> Basic Component; LCSC C55098625 -> C17477; Manufacturer (none) -> UNI-ROYAL(Uniroyal Elec); Minimum Qty (none) -> 20; Operating Temperature Range (none) -> -55°C~+155°C; Overload Voltage (Max) (none) -> 150V; Part (none) -> 0805W8F0000T5E; Power(Watts) (none) -> 125mW; Price (none) -> 0.005USD; Process (none) -> SMT; Resistance (none) -> 0Ω; Stock (none) -> 7792489; Temperature Coefficient (none) -> ±800ppm/°C; Tolerance (none) -> ±1%; Type (none) -> Thick Film Resistors
- R34, R54, R55, R56, R57, R58: symbol PCM_JLCPCB-Resistors_1:0805,10kΩ -> PCM_JLCPCB-Resistors:0805,10kΩ
- U4: LCSC (none) -> C2873264; LCSC  C2873264 -> (none)
Connections:
- net CHG_OUT_POS: now also Q6.1 (S), Q6.2 (S), Q6.3 (S); no longer Q6.5 (D)
- net CTRL_5V: now also D8.2 (VDD)
- net HO1: now also M1.4 (G), TP6.1
- net HO2: now also TP8.1
- net LO1: now also TP7.1
- net LO2: now also TP9.1
- net PGND: no longer C25.1, C26.1, R28.2, R29.2, R30.2, R31.2, R33.2, U6.28 (PGND)
- net PV_IN_POS: now also C21.1, C30.1, C8.1, M1.5 (D)
- net PWR_NEG: now also C25.1, C26.1, R28.2, R29.2, R30.2, R31.2, R33.2, U6.28 (PGND), C33.1, C8.2
- net SRC: now also Q6.5 (D); no longer Q6.1 (S), Q6.2 (S), Q6.3 (S)
- net SW_1: now also M1.1 (S), M1.2 (S), M1.3 (S), TP10.1
- net SW_2: now also TP11.1
- net U6_VCC2: no longer D8.2 (VDD)
- net V_out: now also C33.2; no longer C21.1, C30.1
- net _CSB_2: no longer L2.1, R22.1
- new net: L2.1, R22.1
Other:
- note removed: "Cout"
- note removed: "Input Caps"
- note removed: "Output Caps"
- moved on the sheet: C19, C52, C7, D1, D5, F2, J3, L2, Q2, Q4, R16, R2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

Commit message: hardware: update Rev1 schematic with 0 ERC errors, BOM, and footprint tables
Parts:
- removed TP10, TP11, TP3, TP4, TP5, TP6, TP7, TP8, TP9: TestPoint_Small, Connector_PinHeader_2.54mm:PinHeader_1x01_P2.54mm_Vertical, symbol Connector:TestPoint_Small
- added C31: 47uF, Capacitor_THT:CP_Radial_D8.0mm_P3.50mm, symbol Device:C
- added J6: 20021121-00010C4LF, digikey-footprints:PinHeader_2x5_P1.27mm, symbol 1My_Basic components:20021121-00010C4LF
- added Q7: 2N7002K, PCM_JLCPCB:Q_SOT-23, symbol PCM_JLCPCB-Transistors:NMOS,2N7002K
- added R46: 82kΩ, PCM_JLCPCB:R_0805, symbol PCM_JLCPCB-Resistors:0805,82kΩ
- added R68: 1.3k, PCM_JLCPCB:R_0805, symbol Device:R
- added R69, R70, R71, R72, R73: 10Ω, PCM_JLCPCB:R_0805, symbol PCM_JLCPCB-Resistors:0805,10Ω
- added R74: 100kΩ, PCM_JLCPCB:R_0805, symbol PCM_JLCPCB-Resistors:0805,100kΩ
- added TP15, TP16, TP17, TP18: 5015, TestPoint:TestPoint_Keystone_5015_Micro_Mini, symbol 1My_Connectors:5015
- C18: value 560uf -> 560uF
- C19, C21, C30: value 47uf -> 47uF; footprint Through Hole,D8xL11.5mm -> Capacitor_THT:C_Radial_D8.0mm_H7.0mm_P3.50mm
- C20: value 180pf -> 180pF; LCSC C2168955 -> C1794
- C23: value 100nf -> 100nF
- C24: value 220nf -> 22nF; LCSC C113853 -> C1710
- C25: value 1.5nf -> 1.5nF; LCSC C2169179 -> C1590
- C26: value 10uf -> 33nF; LCSC C161255 -> C1738
- C3: value 100uf -> 100uF
- C49, C50: LCSC C107115 -> C1798
- C7: value 1uf 100v -> 2.2uF; footprint PCM_JLCPCB:C_0805 -> PCM_JLCPCB:C_1206; Attrition Qty (none) -> 8; Capacitance (none) -> 2.2uF; Category (none) -> Capacitors,Multilayer Ceramic Capacitors MLCC - SMD/SMT; Class (none) -> Basic Component; LCSC C6119946 -> C50254; Manufacturer (none) -> Samsung Electro-Mechanics; Minimum Qty (none) -> 5; Part (none) -> CL31B225KBHNNNE; Price (none) -> 0.032USD; Process (none) -> SMT; Stock (none) -> 180873; Temperature Coefficient (none) -> X7R; Tolerance (none) -> ±10%; Voltage Rated (none) -> 50V
- D10, D6, D7: Attrition Qty (none) -> 10; Category (none) -> Diodes,Schottky Barrier Diodes (SBD); Class (none) -> Basic Component; Forward Voltage (Vf@If) (none) -> 600mV@1A; Manufacturer (none) -> Guangdong Hottech; Minimum Qty (none) -> 20; Part (none) -> 1N5819WS; Price (none) -> 0.013USD; Process (none) -> SMT; Rectified Current (none) -> 1A; Reverse Voltage (Vr) (none) -> 40V; Stock (none) -> 1836556
- F1: value Fuse_TD_10A_5x25_63VDC_MIN -> Fuse
- J1: value Solar In -> Screw_Terminal_01x02
- J3: value Battery Bus -> Screw_Terminal_01x02
- J4: value JTAG -> Conn_01x04
- J5: value Fan -> Conn_01x03_Socket
- L2: value 3.3uh -> L; LCSC C2638566 -> C49308530; LCSC  C49308530 -> (none)
- L3: value 68uh -> L
- Q5, Q6: value CSD18563Q5A -> BSC040N10NS5; symbol Transistor_FET:CSD18563Q5A -> Transistor_FET:BSC040N10NS5; LCSC C86513 -> C534334
- R1, R2, R32, R38, R40, R43, R67: LCSC C149504 -> C17416
- R10, R61, R7: LCSC C4328 -> C17523
- R11, R39: LCSC C17630 -> C17650
- R12: LCSC C17772 -> C17730
- R14: LCSC C17629 -> C17651
- R15: LCSC C17604 -> C17537
- R17: LCSC C21437 -> C2933470
- R18, R3: LCSC (none) -> C3000581; LCSC  C3000581 -> (none)
- R19, R34, R36, R47, R48, R50, R53, R54, R55, R56, R57, R58, R59, R6: LCSC C17414 -> C17415
- R20: value 499kΩ -> 499k; LCSC C17721 -> C119857
- R21: LCSC C2988924 -> C119830
- R23: LCSC C17819 -> C17743
- R24, R62: LCSC C27834 -> C17700
- R26, R27, R4, R41, R65: LCSC C17415 -> C17414
- R28: footprint PCM_JLCPCB:R_0603 -> PCM_JLCPCB:R_0805; LCSC C863146 -> C119851
- R29: LCSC C2077356 -> C119842
- R30: LCSC C1854698 -> C119848
- R31: value 2.43K -> 2.43k; LCSC C54532105 -> C119853
- R33, R49, R63, R64: LCSC C17477 -> C17888
- R35, R9: LCSC C17501 -> C17497
- R37, R66: value 2.2M -> 2.2MΩ; LCSC C26113 -> C17539
- R42: value 10Ω -> 1kΩ; symbol PCM_JLCPCB-Resistors:0805,10Ω -> PCM_JLCPCB-Resistors:0805,1kΩ; Attrition Qty 6 -> 10; LCSC C17415 -> C17513; Part 0805W8F100JT5E -> 0805W8F1001T5E; Resistance 10Ω -> 1kΩ; Stock 3283689 -> 7431283; Temperature Coefficient ±200ppm/°C -> ±100ppm/°C
- R51: LCSC C17530 -> C17546
- R60: LCSC C4310 -> C17515
- R8: LCSC C17593 -> C17547
- U1: value STM32F411CEU6 -> STM32G431CBU6; Check_prices https://www.snapeda.com/parts/STM32F411CEU6/STMicroelectron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 -> https://www.snapeda.com/parts/STM32G431CBU6/STMicroelectron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; LCSC C529356 -> (none); MP STM32F411CEU6 -> STM32G431CBU6; Purchase-URL https://www.snapeda.com/api/url_track_click_mouser/?manufac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 -> https://www.snapeda.com/api/url_track_click_mouser/?unipart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; SnapEDA_Link https://www.snapeda.com/parts/STM32F411CEU6/STMicroelectron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 -> https://www.snapeda.com/parts/STM32G431CBU6/STMicroelectron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
- U10: footprint PCM_JLCPCB:SOT-363_SC-70-6 -> INA213AIDCKR:SOT65P210X110-6N
- U2: footprint 113991054:MODULE_113991054 -> 1My_Parts_ MPUs:ESP32 C3 mini
- U4: value LM5163DDAR -> LM5163
- U5: LCSC (none) -> C114569
- U6: footprint Package_DFN_QFN:Texas_RHA0040B_VQFN-40-1EP_6x6mm_P0.5mm_EP4.15x4.15mm -> digikey-footprints:VFQFN-40-1EP_6x6mm
- U7: footprint 1My_Parts_ ICs:Humidity sensor -> AHT20:PSON100P300X300X110-6N
- U8: value (none) -> SSD1306_OLED
Connections:
- net PGND is gone; now on net PWR_NEG: C27.2, C46.2
- net CTRL_3V3: now also R34.1, R74.1, TP17.1; no longer R34.2
- net CTRL_5V: now also TP18.1
- net HO1: now also J6.1, R69.1; no longer U6.24 (HO1)
- net HO2: now also J6.3, R71.1; no longer U6.32 (HO2)
- net I2C CLK: now also J6.2
- net I2C DATA: now also J6.4
- net LO1: now also J6.5, R70.1; no longer U6.27 (LO1)
- net LO2: now also J6.7, R72.1; no longer U6.30 (LO2)
- net PV_IN_POS: now also C31.1, TP16.1
- net PWR_NEG: now also C31.2, Q7.2 (S), R46.2, TP15.1; no longer R32.2
- net SW_1: now also J6.9; no longer R22.3, R26.1
- net SW_2: now also J6.10
- net U6_FLT: now also R34.2; no longer R34.1
- net U6_VCC2: now also R32.1, J6.6
- net V_out: now also R16.1; no longer R16.3, R16.4, R64.2, U10.4 (IN+)
- net V_out_sense: now also R16.4; no longer R16.1, R16.2, R63.2, U10.5 (IN-)
- net _Undervoltage Feedback: now also J6.8, Q7.3 (D)
- net CTRL_EN_CHG: now reaches U1.25 (PB12)
- net CTRL_EN_CHG: now also R73.1
- new net: R69.2, U6.24 (HO1)
- new net: Q7.1 (G), R73.2, R74.2
- new net: R72.2, U6.30 (LO2)
- new net: R71.2, U6.32 (HO2)
- new net: R70.2, U6.27 (LO1)
- new net: R46.1, R68.1
- new net: R68.2, U6.16 (ILIMCOMP_ISET)
- new net: R32.2, U6.7 (MODE)
- new net V_out_SNS_N: R16.3, R63.2, U10.5 (IN-)
- new net V_out_SNS_P : R16.2, R64.2, U10.4 (IN+)
- new net _CSA_2: R22.3, R26.1
- no-connect marks 52 -> 51
Other:
- moved on the sheet: C22, C23, C28, D5, F2, M4, R16, R2, R26, R27, R32, R34

Commit message: handoff: save local Rev1 work for laptop
Parts:
- removed J5: Conn_01x03_Socket, Connector_PinHeader_2.54mm:PinHeader_1x03_P2.54mm_Vertical, symbol Connector:Conn_01x03_Socket
- added D11: WS2812B, PCM_JLCPCB:LED-SMD_4P-L1.6-W1.5_XL-1615RGBC-WS2812B, symbol PCM_JLCPCB-Extended:LED, WS2812B, 1615
- added J7: Fan, Connector_PinHeader_2.54mm:PinHeader_1x03_P2.54mm_Vertical, symbol Connector:Conn_01x03_Pin
- F1, F2: value Fuse -> 3522-2; footprint Fuse:Fuseholder_Littelfuse_100_series_5x25mm -> 1My_Parts_ Passive:3522-2_KEY; symbol Device:Fuse -> 1_Phil's Lib of symbols:3522-2
Connections:
- net BAT_BUS_POS: now also F2.1
- net BTN_RT_N: now also U1.39 (PC10); no longer U1.3 (PC14-OSC32_IN)
- net CHG_OUT_POS: now also F2.3, F2.4, Q6.5 (D), J7.3 (Pin_3); no longer F2.1, Q6.1 (S), Q6.2 (S), Q6.3 (S)
- net CTRL_5V: now also D11.2 (VDD)
- net PV_IN_POS: now also Q4.5 (D); no longer Q4.D
- net PV_IN_POS_FUSED: now also F1.2, Q4.1 (S), Q4.2 (S); no longer Q4.S
- net PV_IN_POS_RAW: now also F1.3, F1.4; no longer F1.2
- net PWR_NEG: now also D11.3 (GND)
- net SRC: now also Q6.1 (S), Q6.2 (S), Q6.3 (S); no longer Q6.5 (D)
- net at D1.2, R42.2: now also Q4.4 (G); no longer Q4.G
- net FAN_TACH: now reaches U1.43 (PB5)
- net FAN_TACH: now also J7.2 (Pin_2)
- net at Q3.3 (D): now also J7.1 (Pin_1)
- net at D8.1 (DOUT): now also D11.4 (DIN)
- no-connect marks 51 -> 49
Other:
- note added: "HB"
- note added: "WiFi"
- moved on the sheet: Q6

Commit message: Save local changes: snapshot of docs, KiCad Rev1, BOM and hardware files
Parts:
- added J8: Conn_01x04, Connector_PinHeader_2.54mm:PinHeader_1x04_P2.54mm_Vertical, symbol Connector_Generic:Conn_01x04
- C19, C21, C30: footprint Capacitor_THT:C_Radial_D8.0mm_H7.0mm_P3.50mm -> Capacitor_THT:CP_Radial_D8.0mm_P3.50mm
- C52: value 100nF -> 220nF; symbol PCM_JLCPCB-Capacitors:0805,100nF -> PCM_JLCPCB-Capacitors:0805,220nF; Capacitance 100nF -> 220nF; LCSC C28233 -> C5378; Part CL21B104KCFNNNE -> CL21B224KBFNNNE; Price 0.009USD -> 0.014USD; Stock 1168020 -> 438651; Voltage Rated 100V -> 50V
- C7: Attrition Qty 8 -> (none); Class Basic Component -> (none); LCSC C50254 -> C577211; Manufacturer Samsung Electro-Mechanics -> YAGEO; Minimum Qty 5 -> (none); Part CL31B225KBHNNNE -> CC1206KKX7R0BB225; Price 0.032USD -> 0.1812USD; Stock 180873 -> 1,013,960; Voltage Rated 50V -> 100V
- D2: value SMBJ60CA -> SMBJ48CA; Breakdown Voltage 78.6V -> (none); LCSC C19077593 -> C151264; Maximum Clamping Voltage 103V -> (none); Number of Lines Dual channel -> (none); Operating Temperature -55°C~+155°C -> (none); Part SMBJ60CA -> SMBJ48CA; Peak Pulse Current (Ipp) 5.83A -> (none); Peak Pulse Power Dissipation (Ppp) 600W -> (none); Price 0.047USD -> 0.1507USD; Reverse Leakage Current (Ir) 5uA -> (none); Reverse Stand-Off Voltage (Vrwm) 64V -> (none); Stock 36646 -> 8,705; Type TVS -> (none); polarity Bidirectional -> (none)
- F1: footprint 1My_Parts_ Passive:3522-2_KEY -> 1My_Parts_ Passive:Automotive fuse holder keystone 3522-2_KEY; LCSC C142864 -> (none); Part - USA TBD -> Keystone 3522-2, sourced via Digikey/Mouser (LCSC does not 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
- F2: footprint 1My_Parts_ Passive:3522-2_KEY -> 1My_Parts_ Passive:Automotive fuse holder keystone 3522-2_KEY; LCSC C142864 -> (none); Part - USA (none) -> Keystone 3522-2, sourced via Digikey/Mouser (LCSC does not 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
- U10: footprint INA213AIDCKR:SOT65P210X110-6N -> PCM_JLCPCB:SOT-363_SC-70-6
- U7: footprint AHT20:PSON100P300X300X110-6N -> 1My_Parts_ ICs:Humidity sensor
Connections:
- net PV_IN_POS_FUSED is gone; now on an unnamed net: D1.1, D2.2, F1.1, F1.2, Q4.1 (S), Q4.2 (S), R35.1, R43.1
- net CTRL_3V3: now also J8.3 (Pin_3)
- net I2C CLK: now also J8.1 (Pin_1)
- net I2C DATA: now also J8.4 (Pin_4)
- net PWR_NEG: now also J8.2 (Pin_2)
- net PV_IN_POS_RAW: no longer names the net of F1.3, F1.4, J1.1 (Pin_1)
